Commit message: update eyeInHand Calibration with Aruco Tag and Charuco

File: src/m6r_description/urdf/camera.xacro (robot description, xacro)
@@ -1,54 +1,58 @@
 <?xml version="1.0"?>
-<robot xmlns:xacro="http://ros.org/wiki/xacro">
-    <material name="red">
-        <color rgba="1 0 0 1"/>
+<robot xmlns:xacro="http://www.ros.org/wiki/xacro">
+    <!--<material name="red">
+      <color rgba="1 0 0 1"/>
+    </material>-->
+    <material name="gray">
+      <color rgba="0.5 0.5 0.5 1"/>
     </material>
+    <joint name="camera_joint" type="fixed">
+	<parent link="wriste_roll"/>
+	<child link="camera_link"/>
+	<origin xyz="0.05 0 0.0" rpy="0 0 0"/>
+    </joint>
     <link name="camera_link">
-        <inertial>
-            <origin xyz="-0.00936000000 -0.00003000000 -0.00273000000" rpy="0 0 0"/>
-            <mass value="0.21970000000"/>
-            <inertia ixx="0.00000429247" ixy="0.00000000000" ixz="0.00000002565"
-                    iyy="0.00000008027" iyz="0.00000000000"
-                    izz="0.00000427339"/>
-        </inertial>
-        <visual>
-            <geometry>
-                <!-- <box size="0.01 0.03 0.03" /> -->
-                <!-- <mesh filename="package://ur_yt_sim/meshes/sensors/camera/kinetic.stl"/> -->
-                <mesh filename="package://m6r_description/meshes/sensors/camera/kinetic.stl"/>
-            </geometry>
-            <material name="red"/>
-        </visual>
-        <collision>
-            <geometry>
-                <!-- <mesh filename="package://ur_yt_sim/meshes/sensors/camera/kinetic.dae"/> -->
-                <mesh filename="package://m6r_description/meshes/sensors/camera/kinetic.dae"/>
-            </geometry>
-        </collision>
+	<visual>
+	    <geometry>
+		<!--<box size="0.010 0.03 0.03"/>-->
+		    <mesh filename="package://m6r_description/meshes/sensors/camera/kinetic.stl"/>
+	    </geometry>
+	    <material name="gray"/>
+	</visual>
     </link>
-    <!-- frames in the center of the camera -->
-    <joint name="camera_joint" type="fixed">
-        <parent link="wriste_roll"/>
-        <child link="camera_link"/>
-        <origin xyz="0 0 0" rpy="0 -1.57 0" />
+    <joint name="camera_optical_joint" type="fixed">
+        <origin xyz="0 0 0" rpy="${-pi/2} 0 ${-pi/2}" />
+        <parent link="camera_link" />
+        <child link="camera_link_optical" />
     </joint>
-    <link name="camera_optical_link"></link>
-    <joint name="camera_optical_joint" type="fixed">
-        <parent link="camera_link"/>
-        <child link="camera_optical_link"/>
-        <origin xyz="0 0 0" rpy="-1.57 0 -1.57" />
-    </joint>
+    <link name="camera_link_optical"></link>
     <gazebo reference="camera_link">
-        <sensor name="camera" type="depth">
-            <pose>0 0 0 0 0 0</pose>
+        <sensor name="depth_camera" type="depth">
             <visualize>true</visualize>
-            <update_rate>10</update_rate>
-            <camera>
-            <horizontal_fov>1.089</horizontal_fov>
-            <image><format>R8G8B8</format><width>640</width><height>480</height></image>
-            <clip><near>0.05</near><far>8</far></clip>
+            <update_rate>30.0</update_rate>
+            <camera name="camera">
+            <horizontal_fov>1.5708</horizontal_fov>
+            <image>
+                <width>640</width>
+                <height>480</height>
+                <format>R8G8B8</format>
+            </image>
+            <clip>
+                <near>0.05</near>
+                <far>10.0</far>
+            </clip>
             </camera>
-            <plugin name="camera_controller" filename="libgazebo_ros_camera.so">
-            <frame_name>camera_optical_link</frame_name>
+            <plugin name="depth_camera_controller" filename="libgazebo_ros_camera.so">
+            <ros>
+                <namespace>/</namespace>
+                <remapping>image_raw:=camera/image_raw</remapping>
+                <remapping>depth/image_raw:=camera/depth_image_raw</remapping>
+                <remapping>camera_info:=camera/camera_info</remapping>
+                <remapping>depth/camera_info:=camera/depth_info</remapping>
+                <remapping>points:=camera/points</remapping>
+            </ros>
+            <frame_name>camera_link_optical</frame_name>
+            <min_depth>0.1</min_depth>
+            <max_depth>10.0</max_depth>
             </plugin>
         </sensor>
