Commit message: udpate camera to correct position

File: src/m6r_description/urdf/camera2.xacro (robot description, xacro)
@@ -1,68 +1,80 @@
 <?xml version="1.0"?>
 <robot xmlns:xacro="http://www.ros.org/wiki/xacro">
-    <!--<material name="red">
-      <color rgba="1 0 0 1"/>
-    </material>-->
     <material name="gray">
-      <color rgba="0.5 0.5 0.5 1"/>
+        <color rgba="0.5 0.5 0.5 1"/>
     </material>
     <joint name="camera_joint" type="fixed">
-	<parent link="wriste_roll"/>
-	<child link="camera_link"/>
-	<origin xyz="0.05 0 0.0" rpy="0 0 0"/>
+        <origin xyz="-0.155 0 -0.059" rpy="0 -0.00015 0"/>
+        <parent link="wriste_roll" />
+        <child link="camera_link" />
     </joint>
     <link name="camera_link">
-	<visual>
-	    <geometry>
-		<!--<box size="0.010 0.03 0.03"/>-->
-		    <mesh filename="package://m6r_description/meshes/sensors/camera/kinetic.stl"/>
-	    </geometry>
-	    <material name="gray"/>
-	</visual>
+        <inertial>
+            <origin xyz="0 0 0" rpy="0 0 0" />
+            <mass value="0.012" />
+            <inertia ixx="0.0001" ixy="0" ixz="0" iyy="0.0001" iyz="0" izz="0.0001" />
+        </inertial>
+        <visual>
+            <origin xyz="0 0 0" rpy="3.14 0 1.57" />
+            <geometry>
+                <mesh filename="package://m6r_description/meshes/m6r_0110/camera.STL" />
+            </geometry>
+            <material name="gray"/>
+        </visual>
+        <collision>
+            <origin xyz="0 0 0" rpy="0 0 0" />
+            <geometry>
+                <box size="0.05 0.03 0.03"/>
+            </geometry>
+        </collision>
     </link>
     <joint name="camera_optical_joint" type="fixed">
-        <origin xyz="0 0 0" rpy="${-pi/2} 0 ${-pi/2}" />
+        <origin xyz="0 0 0" rpy="1.57 0.0 0.0" />
         <parent link="camera_link" />
         <child link="camera_link_optical" />
     </joint>
-    <link name="camera_link_optical"></link>
+    <link name="camera_link_optical">
+        <inertial>
+            <mass value="0.001" />
+            <inertia ixx="0.0001" ixy="0" ixz="0" iyy="0.0001" iyz="0" izz="0.0001" />
+        </inertial>
+    </link>
     <gazebo reference="camera_link">
-        <!--<material>Gazebo/Red</material>-->
         <material>Gazebo/Gray</material>
-	<sensor name="camera" type="camera">
-    	    <pose> 0 0 0 0 0 0 </pose>
-    	    <visualize>true</visualize>
-    	    <update_rate>10</update_rate>
-	    <camera>
-	        <horizontal_fov>1.089</horizontal_fov>
-	        <image>
-		    <format>R8G8B8</format>
-		    <width>640</width>
-		    <height>480</height>
-	        </image>
-	        <clip>
-		    <near>0.05</near>
-		    <far>8.0</far>
-	        </clip>
-	       <lens>
-      		<intrinsics>
-        	  <fx>500</fx>
-        	  <fy>500</fy>
-        	  <cx>320</cx>
-        	  <cy>240</cy>
-        	  <s>0</s>
-      		</intrinsics>
-    	       </lens>
-	    </camera>
-	    <plugin name="camera_controller" filename="libgazebo_ros_camera.so">
-			<ros>
-				<namespace>/</namespace>
-				<remapping>image_raw:=camera/image_raw</remapping>
-				<remapping>camera_info:=camera/camera_info</remapping>
-			</ros>
-			<frame_name>camera_link_optical</frame_name>
-			<hack_baseline>0.07</hack_baseline>
-		</plugin>
-	</sensor>
+        <sensor name="camera" type="camera">
+            <pose>0 0 0 0 0 0</pose>
+            <visualize>true</visualize>
+            <update_rate>10</update_rate>
+            <camera>
+                <horizontal_fov>1.089</horizontal_fov>
+                <image>
+                    <format>R8G8B8</format>
+                    <width>640</width>
+                    <height>480</height>
+                </image>
+                <clip>
+                    <near>0.05</near>
+                    <far>8.0</far>
+                </clip>
+                <lens>
+                    <intrinsics>
+                        <fx>500</fx>
+                        <fy>500</fy>
+                        <cx>320</cx>
+                        <cy>240</cy>
+                        <s>0</s>
+                    </intrinsics>
+                </lens>
+            </camera>
+            <plugin name="camera_controller" filename="libgazebo_ros_camera.so">
+                <ros>
+                    <namespace>/</namespace>
+                    <remapping>image_raw:=camera/image_raw</remapping>
+                    <remapping>camera_info:=camera/camera_info</remapping>
+                </ros>
+                <frame_name>camera_link_optical</frame_name>
+                <hack_baseline>0.07</hack_baseline>
+            </plugin>
+        </sensor>
     </gazebo>
 </robot>
