Commit message: modified the decription and bringup pkgs to add gazebo simulation and camera image

File: src/m6r_description/urdf/m6r.urdf.xacro (robot description, xacro)
@@ -1,5 +1,17 @@
 <?xml version="1.0"?>
 <robot xmlns:xacro="http://wiki.ros.org/xacro" name="m6r">
-    <xacro:include filename="m6r.xacro" />
-    <xacro:include filename="m6r.ros2_control.xacro"/>
+    <!-- <xacro:include filename="m6r.xacro" /> -->
+    <!-- <xacro:include filename="m6r_0110.xacro"/>
+    <xacro:include filename="m6r.ros2_control.xacro"/> -->
+    <!-- <xacro:include filename="camera.xacro"/> -->
+    <link name="world"/>
+    <joint name="world_to_base" type="fixed">
+        <parent link="world"/>
+        <child link="base_link"/>
+        <origin xyz="0 0 0" rpy="0 0 0"/>
+    </joint>
+    <xacro:include filename="m6r_0110.xacro"/>
+    <xacro:include filename="gazebo.ros2_control.xacro"/>
+    <xacro:include filename="m6r.gazebo.xacro"/>
+    <xacro:include filename="camera2.xacro"/>
 </robot>

File: src/m6r_mod_moveit_config2/config/m6r.urdf.xacro (robot description, xacro)
@@ -3,5 +3,5 @@
     <xacro:arg name="initial_positions_file" default="initial_positions.yaml" />
     <!-- Import m6r urdf file -->
-    <xacro:include filename="$(find m6r_description)/urdf/m6r.urdf" />
+    <xacro:include filename="$(find m6r_description)/urdf/m6r_0110.urdf" />
     <!-- Import control_xacro -->
     <xacro:include filename="m6r.ros2_control.xacro" />

Commit message: update world frame calibration with both aruco and charuco, update readme to generate the gazebo model of makers

File: src/m6r_description/urdf/m6r.urdf.xacro (robot description, xacro)
@@ -5,9 +5,10 @@
     <xacro:include filename="m6r.ros2_control.xacro"/> -->
     <!-- <xacro:include filename="camera.xacro"/> -->
+        <!-- <origin xyz="0.4 0.2 -0.07" rpy="0 0 0"/> -->
     <link name="world"/>
     <joint name="world_to_base" type="fixed">
         <parent link="world"/>
         <child link="base_link"/>
-        <origin xyz="0 0 0" rpy="0 0 0"/>
+        <origin xyz="0 0 -0.07" rpy="0 0 0"/>
     </joint>
     <xacro:include filename="m6r_0110.xacro"/>
